Commit message: Made a bot with a front and back leg, and a torso.

File: body.urdf (robot description, URDF)
Before this commit: robot robot, 5 links, 4 joints
Links:
- removed link Link0
- removed link Link1
- removed link Link2
- removed link Link3
- removed link Link4
- added link BackLeg, mass 1; collision box size=1 1 1; visual box size=1 1 1
- added link FrontLeg, mass 1; collision box size=1 1 1; visual box size=1 1 1
- added link Torso, mass 1; collision box size=1 1 1; visual box size=1 1 1
Joints:
- removed joint Link0_Link1
- removed joint Link1_Link2
- removed joint Link2_Link3
- removed joint Link3_Link4
- added joint Torso_BackLeg: type revolute, parent Torso, child BackLeg, origin xyz=1 0 1 rpy=0 0 0, axis 0 1 0, limit lower=-3.14159 upper=3.14159 effort=0.0 velocity=0.0
- added joint Torso_FrontLeg: type revolute, parent Torso, child FrontLeg, origin xyz=2 0 1 rpy=0 0 0, axis 0 1 0, limit lower=-3.14159 upper=3.14159 effort=0.0 velocity=0.0

Commit message: Created robot with torso, frontleg, and backleg.

File: body.urdf (robot description, URDF)
Before this commit: robot robot, 7 links, 6 joints
Links:
- removed link Link0
- removed link Link1
- removed link Link2
- removed link Link3
- removed link Link4
- removed link Link5
- removed link Link6
- added link BackLeg, mass 1; collision box size=1 1 1; visual box size=1 1 1
- added link FrontLeg, mass 1; collision box size=1 1 1; visual box size=1 1 1
- added link Torso, mass 1; collision box size=1 1 1; visual box size=1 1 1
Joints:
- removed joint Link0_Link1
- removed joint Link1_Link2
- removed joint Link2_Link3
- removed joint Link3_Link4
- removed joint Link4_Link5
- removed joint Link5_Link6
- added joint Torso_BackLeg: type revolute, parent Torso, child BackLeg, origin xyz=0.5 0 2.0 rpy=0 0 0, axis 0 1 0, limit lower=-3.14159 upper=3.14159 effort=0.0 velocity=0.0
- added joint Torso_FrontLeg: type revolute, parent Torso, child FrontLeg, origin xyz=-0.5 0 2.0 rpy=0 0 0, axis 0 1 0, limit lower=-3.14159 upper=3.14159 effort=0.0 velocity=0.0

Commit message: Swapped position of front and back leg. Printing touch sensor values to the console.

File: body.urdf (robot description, URDF)
Before this commit: robot robot, 3 links, 2 joints
Joints:
- joint Torso_BackLeg: origin xyz=0.5 0 2.0 rpy=0 0 0 -> xyz=-0.5 0 2.0 rpy=0 0 0
- joint Torso_FrontLeg: origin xyz=-0.5 0 2.0 rpy=0 0 0 -> xyz=0.5 0 2.0 rpy=0 0 0

Commit message: Fixed an issue where robot wasn't starting at ground level making the leg sensor neurons output a 0 instead of a 2.0.

File: body.urdf (robot description, URDF)
Before this commit: robot robot, 3 links, 2 joints
Joints:
- joint Torso_BackLeg: origin xyz=-0.5 0 2.0 rpy=0 0 0 -> xyz=-0.5 0 1.0 rpy=0 0 0
- joint Torso_FrontLeg: origin xyz=0.5 0 2.0 rpy=0 0 0 -> xyz=0.5 0 1.0 rpy=0 0 0

Commit message: Moved the links around the match the picture. Completed front-leg.

File: body.urdf (robot description, URDF)
Before this commit: robot robot, 3 links, 2 joints
Links:
- link FrontLeg: geometry collision box size=0.2 1 0.2; visual box size=0.2 1 0.2
Joints:
- joint Torso_BackLeg: origin xyz=-0.5 0 1.0 rpy=0 0 0 -> xyz=-0.5 0 1.5 rpy=0 0 0
- joint Torso_FrontLeg: origin xyz=0.5 0 1.0 rpy=0 0 0 -> xyz=0.5 0 1.5 rpy=0 0 0

Commit message: Finished the backleg.

File: body.urdf (robot description, URDF)
Before this commit: robot robot, 3 links, 2 joints
Links:
- link BackLeg: geometry collision box size=0.2 1 0.2; visual box size=0.2 1 0.2
Joints:
- joint Torso_BackLeg: axis 0 1 0 -> 1 0 0; origin xyz=-0.5 0 1.5 rpy=0 0 0 -> xyz=0 -0.5 1 rpy=0 0 0
- joint Torso_FrontLeg: axis 0 1 0 -> 1 0 0; origin xyz=0.5 0 1.5 rpy=0 0 0 -> xyz=0 0.5 1 rpy=0 0 0

Commit message: Added left leg

File: body.urdf (robot description, URDF)
Before this commit: robot robot, 3 links, 2 joints
Links:
- added link LeftLeg, mass 1; collision box size=1 0.2 0.2; visual box size=1 0.2 0.2
Joints:
- added joint Torso_LeftLeg: type revolute, parent Torso, child LeftLeg, origin xyz=-0.5 0 1 rpy=0 0 0, axis 0 1 0, limit lower=-3.14159 upper=3.14159 effort=0.0 velocity=0.0

Commit message: Added right leg

File: body.urdf (robot description, URDF)
Before this commit: robot robot, 4 links, 3 joints
Links:
- added link RightLeg, mass 1; collision box size=1 0.2 0.2; visual box size=1 0.2 0.2
Joints:
- added joint Torso_RightLeg: type revolute, parent Torso, child RightLeg, origin xyz=0.5 0 1 rpy=0 0 0, axis 0 1 0, limit lower=-3.14159 upper=3.14159 effort=0.0 velocity=0.0

Commit message: Added lower limbs to quadruped

File: body.urdf (robot description, URDF)
Before this commit: robot robot, 5 links, 4 joints
Links:
- added link BackLowerLeg, mass 1; collision box size=0.2 0.2 1; visual box size=0.2 0.2 1
- added link FrontLowerLeg, mass 1; collision box size=0.2 0.2 1; visual box size=0.2 0.2 1
- added link LeftLowerLeg, mass 1; collision box size=0.2 0.2 1; visual box size=0.2 0.2 1
- added link RightLowerLeg, mass 1; collision box size=0.2 0.2 1; visual box size=0.2 0.2 1
Joints:
- added joint BackLeg_BackLowerLeg: type revolute, parent BackLeg, child BackLowerLeg, origin xyz=0 -1 1 rpy=0 0 0, axis 0 0 1, limit lower=-3.14159 upper=3.14159 effort=0.0 velocity=0.0
- added joint FrontLeg_FrontLowerLeg: type revolute, parent FrontLeg, child FrontLowerLeg, origin xyz=0 1 1 rpy=0 0 0, axis 0 0 1, limit lower=-3.14159 upper=3.14159 effort=0.0 velocity=0.0
- added joint LeftLeg_LeftLowerLeg: type revolute, parent LeftLeg, child LeftLowerLeg, origin xyz=-1 0 1 rpy=0 0 0, axis 0 0 1, limit lower=-3.14159 upper=3.14159 effort=0.0 velocity=0.0
- added joint RightLeg_RightLowerLeg: type revolute, parent RightLeg, child RightLowerLeg, origin xyz=1 0 1 rpy=0 0 0, axis 0 0 1, limit lower=-3.14159 upper=3.14159 effort=0.0 velocity=0.0

Commit message: Fixed problem with the link and joint coordinates. Finished quadruped.

File: body.urdf (robot description, URDF)
Before this commit: robot robot, 9 links, 8 joints
Joints:
- joint BackLeg_BackLowerLeg: axis 0 0 1 -> 1 0 0; origin xyz=0 -1 1 rpy=0 0 0 -> xyz=0 -1 0 rpy=0 0 0
- joint FrontLeg_FrontLowerLeg: axis 0 0 1 -> 1 0 0; origin xyz=0 1 1 rpy=0 0 0 -> xyz=0 1 0 rpy=0 0 0
- joint LeftLeg_LeftLowerLeg: axis 0 0 1 -> 0 1 0; origin xyz=-1 0 1 rpy=0 0 0 -> xyz=-1 0 0 rpy=0 0 0
- joint RightLeg_RightLowerLeg: axis 0 0 1 -> 0 1 0; origin xyz=1 0 1 rpy=0 0 0 -> xyz=1 0 0 rpy=0 0 0

Commit message: Created links and joints for atlas robot.

File: body.urdf (robot description, URDF)
Before this commit: robot robot, 9 links, 8 joints
Links:
- removed link BackLeg
- removed link BackLowerLeg
- removed link FrontLeg
- removed link FrontLowerLeg
- added link Head, mass 1; collision box size=0.4 1 0.8; visual box size=0.4 1 0.8
- added link LeftArm, mass 1; collision box size=0.4 0.4 1; visual box size=0.4 0.4 1
- added link LeftLowerArm, mass 1; collision box size=0.2 0.2 1.2; visual box size=0.2 0.2 1.2
- added link RightArm, mass 1; collision box size=0.4 0.4 1; visual box size=0.4 0.4 1
- added link RightLowerArm, mass 1; collision box size=0.2 0.2 1.2; visual box size=0.2 0.2 1.2
- link LeftLeg: geometry collision box size=0.4 0.4 1; visual box size=0.4 0.4 1
- link RightLeg: geometry collision box size=0.4 0.4 1; visual box size=0.4 0.4 1
- link Torso: geometry collision box size=0.8 1 2; visual box size=0.8 1 2
Joints:
- removed joint BackLeg_BackLowerLeg
- removed joint FrontLeg_FrontLowerLeg
- removed joint Torso_BackLeg
- removed joint Torso_FrontLeg
- added joint LeftArm_LeftLowerArm: type revolute, parent LeftArm, child LeftLowerArm, origin xyz=0 0 -1 rpy=0 0 0, axis 0 1 0, limit lower=-3.14159 upper=3.14159 effort=0.0 velocity=0.0
- added joint Left_Torso: type revolute, parent LeftLeg, child Torso, origin xyz=0 0.5 2.1 rpy=0 0 0, axis 0 1 0, limit lower=-3.14159 upper=3.14159 effort=0.0 velocity=0.0
- added joint RightArm_RightLowerArm: type revolute, parent RightArm, child RightLowerArm, origin xyz=0 0 -1 rpy=0 0 0, axis 0 1 0, limit lower=-3.14159 upper=3.14159 effort=0.0 velocity=0.0
- added joint Torso_Head: type revolute, parent Torso, child Head, origin xyz=0 0 3.25 rpy=0 0 0, axis 1 0 0, limit lower=-3.14159 upper=3.14159 effort=0.0 velocity=0.0
- added joint Torso_LeftArm: type revolute, parent Torso, child LeftArm, origin xyz=0 -0.7 4 rpy=0 0 0, axis 0 1 0, limit lower=-3.14159 upper=3.14159 effort=0.0 velocity=0.0
- added joint Torso_RightArm: type revolute, parent Torso, child RightArm, origin xyz=0 0.7 4 rpy=0 0 0, axis 0 1 0, limit lower=-3.14159 upper=3.14159 effort=0.0 velocity=0.0
- joint LeftLeg_LeftLowerLeg: origin xyz=-1 0 0 rpy=0 0 0 -> xyz=0 0 -1 rpy=0 0 0
- joint RightLeg_RightLowerLeg: origin xyz=1 0 0 rpy=0 0 0 -> xyz=0 0 -1 rpy=0 0 0
- joint Torso_LeftLeg: origin xyz=-0.5 0 1 rpy=0 0 0 -> xyz=0 0.5 2.1 rpy=0 0 0
- joint Torso_RightLeg: origin xyz=0.5 0 1 rpy=0 0 0 -> xyz=0 -0.5 2.1 rpy=0 0 0

Commit message: Changed robot.py's Get_Fitness method to allow the robot to move in response to balance as well.

File: body.urdf (robot description, URDF)
Before this commit: robot robot, 10 links, 10 joints
Joints:
- removed joint Left_Torso

Commit message: Removed the arms in this git branch. The arms definetly make it easier for the robot to maintain its balance.

File: body.urdf (robot description, URDF)
Before this commit: robot robot, 10 links, 9 joints
Links:
- removed link LeftArm
- removed link LeftLowerArm
- removed link RightArm
- removed link RightLowerArm
Joints:
- removed joint LeftArm_LeftLowerArm
- removed joint RightArm_RightLowerArm
- removed joint Torso_LeftArm
- removed joint Torso_RightArm
